File: testPCB/switchedPhaseShift.kicad_pcb (KiCad board)
At the start: 4 copper layers, 30 x 85 mm, 83 parts, among them J1 Conn_Coaxial, J10 Conn_Coaxial, J11 Conn_Coaxial, J12 Conn_Coaxial, J13 Conn_Coaxial, J14 Conn_Coaxial, J15 Conn_Coaxial, J16 Conn_Coaxial, J17 Conn_Coaxial, J18 Conn_Coaxial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

Commit message: minor design fixes for test pcb
- gnd plane should not be on f.cu
- remove solder mask on f.cu over antenna
- add DC block capacitors on board outputs to VNA (to J1 and J18)
Parts:
- added C29: 8.2p, Capacitor_SMD:C_0201_0603Metric_Pad0.64x0.40mm_HandSolder, B.Cu at (133.3, 116.3)
- added C30: 8.2p, Capacitor_SMD:C_0201_0603Metric_Pad0.64x0.40mm_HandSolder, B.Cu at (130.8, 156.2)
- moved J1 0.22 mm to (133.3, 123.4)
Connections:
- J1 pad 1: /SL_PhaseShift1/RF_OUT2 -> Net-(J1-In)
- J18 pad 1: /VectorModulator/RF_OUT -> Net-(J18-In)
Routing:
- net Net-(J1-In): track 0.00 -> 5.66 mm
- net /VectorModulator/RF_OUT: track 6.42 -> 2.57 mm
- net /SL_PhaseShift1/RF_OUT2: track 4.03 -> 0.91 mm
- net Net-(J18-In): track 0.00 -> 3.04 mm
- removed copper zone on F.Cu, net GND

Commit message: generate gerbers
Parts:
- removed TP6: TB_IBBN, TestPoint:TestPoint_Pad_1.5x1.5mm
- added IBBN: TB_IBBN, TestPoint:TestPoint_Pad_1.5x1.5mm, B.Cu at (140.1, 154.0)
- renumbered TP5 to IBBP, J18 to IQ_OUT, TP8 to QBBN, TP7 to QBBP
Routing:
- net GND: track 0.00 -> 72.4 mm, vias 4 -> 53
- net /SL_PhaseShift1/C4: track 36.1 -> 35.1 mm
Other:
- board text added: "+5V"
- board text added: "+VS"
- board text added: "Ant_In"
- board text added: "C1"
- board text added: "C2"
- board text added: "C3"
- board text added: "C4"
- board text added: "C5"
- board text added: "GND"
- board text added: "IQ_In"
- board text added: "Line"
- board text added: "Reflect"
- board text added: "T_Junc"
- board text added: "Trace"
- board text added: "Wilkinson"
