File: testPCB/Amplifier_SBB5089Z.kicad_sch (KiCad schematic)
At the start: 6 parts, among them U15 SBB5089Z

Commit message: 4 element phase shifter designed
Parts:
- C11: value 68p -> 100p; footprint Capacitor_SMD:C_0201_0603Metric_Pad0.64x0.40mm_HandSolder -> Capacitor_SMD:C_0603_1608Metric_Pad1.08x0.95mm_HandSolder
Changed lines of the file:
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@@
 			)
 		)
-		(property "Value" "68p"
+		(property "Value" "100p"
 			(at 107.95 66.0335 0)
 			(effects
@@
 			)
 		)
-		(property "Footprint" "Capacitor_SMD:C_0201_0603Metric_Pad0.64x0.40mm_HandSolder"
+		(property "Footprint" "Capacitor_SMD:C_0603_1608Metric_Pad1.08x0.95mm_HandSolder"
 			(at 105.41 64.77 0)
 			(effects
