File: testPCB/SL_PhaseShift.kicad_sch (KiCad schematic)
At the start: 6 parts

Commit message: 4 element phase shifter designed
Connections:
- net Bottom path is short path: now reaches U4.4 (RF1), U5.2 (RF3)
Other:
- note added: "Top path is long path"
- note added: "V1 High = RF1 to RF4, RF2 to RF3 V1 Low = RF1 to RF3, RF2 to RF4"
- note removed: "V1 High = ANT1 to RX, ANT2 to TX V1 Low = ANT1 to TX, ANT2 to RX V1 = V2'"
Changed lines of the file:
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@@
 	(generator_version "9.0")
 	(paper "A4")
-	(text "V1 High = ANT1 to RX, ANT2 to TX\nV1 Low = ANT1 to TX, ANT2 to RX\nV1 = V2'\n"
+	(text "Top path is long path\n"
+		(exclude_from_sim no)
+		(at 81.026 59.944 0)
+		(effects
+			(font
+				(size 1.27 1.27)
+			)
+		)
+	)
+	(text "V1 High = RF1 to RF4, RF2 to RF3\nV1 Low = RF1 to RF3, RF2 to RF4\n"
 		(exclude_from_sim no)
 		(at 63.246 106.934 0)
@@
 		(effects
 			(font
+				(size 1.27 1.27)
+			)
+			(justify left bottom)
+		)
+	)
+	(label "Bottom path is short path"
+		(at 72.39 90.17 0)
+		(effects
+			(font
