File: testPCB/Vector_Modulator_TestBoard.kicad_sch (KiCad schematic)
At the start: 27 parts, among them U10 AMS1117, U11 TLV2372, U9 ADL5375-15ACPZ-WP

Commit message: 4 element phase shifter designed
Parts:
- C24, C25: value 100pF -> 100p
Changed lines of the file:
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@@
 			)
 		)
-		(property "Value" "100pF"
+		(property "Value" "100p"
 			(at 151.13 114.2935 0)
 			(effects
@@
 			)
 		)
-		(property "Value" "100pF"
+		(property "Value" "100p"
 			(at 151.13 127.0062 0)
 			(effects
