File: testPCB/switchedPhaseShift.kicad_sch (KiCad schematic)
At the start: 38 parts, among them J1 Conn_Coaxial, J10 Conn_Coaxial, J11 Conn_Coaxial, J12 Conn_Coaxial, J13 Conn_Coaxial, J14 Conn_Coaxial, J15 Conn_Coaxial, J16 Conn_Coaxial, J17 Conn_Coaxial, J18 Conn_Coaxial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

Commit message: minor design fixes for test pcb
- gnd plane should not be on f.cu
- remove solder mask on f.cu over antenna
- add DC block capacitors on board outputs to VNA (to J1 and J18)
Parts:
- added C29, C30: 8.2p, Capacitor_SMD:C_0201_0603Metric_Pad0.64x0.40mm_HandSolder, symbol Device:C_Small
Connections:
- net SL_PhaseShift1/RF_OUT2: now also C29.2; no longer J1.1 (In)
- net VectorModulator/RF_OUT: now also C30.2; no longer J18.1 (In)
- new net: C29.1, J1.1 (In)
- new net: C30.1, J18.1 (In)
Other:
- note removed: "Unsure what to do with this oscillator You figure out how you want to test it"
- moved on the sheet: J1, J18
Changed lines of the file:
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@@
 		)
 	)
-	(text "Unsure what to do with this oscillator\nYou figure out how you want to test it"
-		(exclude_from_sim no)
-		(at 50.038 4.826 0)
-		(effects
-			(font
-				(size 3 3)
-				(thickness 0.6)
-				(bold yes)
-			)
-		)
-	)
 	(junction
 		(at 66.04 52.07)
@@
 	(wire
 		(pts
+			(xy 93.98 129.54) (xy 102.87 129.54)
+		)
+		(stroke
+			(width 0)
+			(type default)
+		)
+	)
+	(wire
+		(pts
 			(xy 17.78 67.31) (xy 17.78 57.15)
 		)
@@
 	(wire
 		(pts
+			(xy 106.68 157.48) (xy 115.57 157.48)
+		)
+		(stroke
+			(width 0)
+			(type default)
+		)
+	)
+	(wire
+		(pts
 			(xy 242.57 35.56) (xy 255.27 35.56)
 		)
@@
 	(wire
 		(pts
+			(xy 107.95 129.54) (xy 116.84 129.54)
+		)
+		(stroke
+			(width 0)
+			(type default)
+		)
+	)
+	(wire
+		(pts
 			(xy 54.61 157.48) (xy 63.5 157.48)
 		)
@@
 	(wire
 		(pts
-			(xy 93.98 129.54) (xy 104.14 129.54)
+			(xy 93.98 157.48) (xy 101.6 157.48)
 		)
 		(stroke
@@
 	(wire
 		(pts
-			(xy 93.98 157.48) (xy 104.14 157.48)
-		)
-		(stroke
-			(width 0)
-			(type default)
-		)
-	)
-	(wire
-		(pts
 			(xy 173.99 67.31) (xy 190.5 67.31)
 		)
@@
 	)
 	(symbol
+		(lib_id "Device:C_Small")
+		(at 105.41 129.54 270)
+		(unit 1)
+		(exclude_from_sim no)
+		(in_bom yes)
+		(on_board yes)
+		(dnp no)
+		(fields_autoplaced yes)
+		(property "Reference" "C29"
+			(at 105.4036 123.19 90)
+			(effects
+				(font
+					(size 1.27 1.27)
+				)
+			)
+		)
+		(property "Value" "8.2p"
+			(at 105.4036 125.73 90)
+			(effects
+				(font
+					(size 1.27 1.27)
+				)
+			)
+		)
+		(property "Footprint" "Capacitor_SMD:C_0201_0603Metric_Pad0.64x0.40mm_HandSolder"
+			(at 105.41 129.54 0)
+			(effects
+				(font
+					(size 1.27 1.27)
+				)
+				(hide yes)
+			)
+		)
+		(property "Datasheet" "~"
+			(at 105.41 129.54 0)
+			(effects
+				(font
+					(size 1.27 1.27)
+				)
+				(hide yes)
+			)
+		)
+		(property "Description" "Unpolarized capacitor, small symbol"
+			(at 105.41 129.54 0)
+			(effects
+				(font
+					(size 1.27 1.27)
+				)
+				(hide yes)
+			)
+		)
+		(pin "2"
+		)
+		(pin "1"
+		)
+		(instances
+			(project "switchedPhaseShift"
+				(path "/1d55951e-8a24-49b3-bfbf-6f2cb30e41cb"
+					(reference "C29")
+					(unit 1)
+				)
+			)
+		)
+	)
+	(symbol
 		(lib_id "power:GND")
 		(at 71.12 52.07 0)
@@
 	)
 	(symbol
+		(lib_id "Device:C_Small")
+		(at 104.14 157.48 270)
+		(unit 1)
+		(exclude_from_sim no)
+		(in_bom yes)
+		(on_board yes)
+		(dnp no)
+		(fields_autoplaced yes)
+		(property "Reference" "C30"
+			(at 104.1336 151.13 90)
+			(effects
+				(font
+					(size 1.27 1.27)
+				)
+			)
+		)
+		(property "Value" "8.2p"
+			(at 104.1336 153.67 90)
+			(effects
+				(font
+					(size 1.27 1.27)
+				)
+			)
+		)
+		(property "Footprint" "Capacitor_SMD:C_0201_0603Metric_Pad0.64x0.40mm_HandSolder"
+			(at 104.14 157.48 0)
+			(effects
+				(font
+					(size 1.27 1.27)
+				)
+				(hide yes)
+			)
+		)
+		(property "Datasheet" "~"
+			(at 104.14 157.48 0)
+			(effects
+				(font
+					(size 1.27 1.27)
+				)
+				(hide yes)
+			)
+		)
+		(property "Description" "Unpolarized capacitor, small symbol"
+			(at 104.14 157.48 0)
+			(effects
+				(font
+					(size 1.27 1.27)
+				)
+				(hide yes)
+			)
+		)
+		(pin "2"
+		)
+		(pin "1"
+		)
+		(instances
+			(project "switchedPhaseShift"
+				(path "/1d55951e-8a24-49b3-bfbf-6f2cb30e41cb"
+					(reference "C30")
+					(unit 1)
+				)
+			)
+		)
+	)
+	(symbol
 		(lib_id "Connector:Conn_Coaxial")
 		(at 49.53 157.48 0)
@@
 	(symbol
 		(lib_id "power:GND")
-		(at 109.22 162.56 0)
+		(at 120.65 162.56 0)
 		(mirror y)
 		(unit 1)
@@
 		(fields_autoplaced yes)
 		(property "Reference" "#PWR025"
-			(at 109.22 168.91 0)
+			(at 120.65 168.91 0)
 			(effects
 				(font
@@
 		)
 		(property "Value" "GND"
-			(at 109.22 167.64 0)
+			(at 120.65 167.64 0)
 			(effects
 				(font
@@
 		)
 		(property "Footprint" ""
-			(at 109.22 162.56 0)
+			(at 120.65 162.56 0)
 			(effects
 				(font
@@
 		)
 		(property "Datasheet" ""
-			(at 109.22 162.56 0)
+			(at 120.65 162.56 0)
 			(effects
 				(font
@@
 		)
 		(property "Description" "Power symbol creates a global label with name \"GND\" , ground"
-			(at 109.22 162.56 0)
+			(at 120.65 162.56 0)
 			(effects
 				(font
@@
 	(symbol
 		(lib_id "power:GND")
-		(at 109.22 134.62 0)
+		(at 121.92 134.62 0)
 		(mirror y)
 		(unit 1)
@@
 		(fields_autoplaced yes)
 		(property "Reference" "#PWR019"
-			(at 109.22 140.97 0)
+			(at 121.92 140.97 0)
 			(effects
 				(font
@@
 		)
 		(property "Value" "GND"
-			(at 109.22 139.7 0)
+			(at 121.92 139.7 0)
 			(effects
 				(font
@@
 		)
 		(property "Footprint" ""
-			(at 109.22 134.62 0)
+			(at 121.92 134.62 0)
 			(effects
 				(font
@@
 		)
 		(property "Datasheet" ""
-			(at 109.22 134.62 0)
+			(at 121.92 134.62 0)
 			(effects
 				(font
@@
 		)
 		(property "Description" "Power symbol creates a global label with name \"GND\" , ground"
-			(at 109.22 134.62 0)
+			(at 121.92 134.62 0)
 			(effects
 				(font
@@
 	(symbol
 		(lib_id "Connector:Conn_Coaxial")
-		(at 109.22 129.54 0)
+		(at 121.92 129.54 0)
 		(unit 1)
 		(exclude_from_sim no)
@@
 		(dnp no)
 		(property "Reference" "J1"
-			(at 113.03 128.5631 0)
+			(at 125.73 128.5631 0)
 			(effects
 				(font
@@
 		)
 		(property "Value" "Conn_Coaxial"
-			(at 113.03 131.1031 0)
+			(at 125.73 131.1031 0)
 			(effects
 				(font
@@
 		)
 		(property "Footprint" "Connector_Coaxial:U.FL_Hirose_U.FL-R-SMT-1_Vertical"
-			(at 109.22 129.54 0)
+			(at 121.92 129.54 0)
 			(effects
 				(font
@@
 		)
 		(property "Datasheet" "~"
-			(at 109.22 129.54 0)
+			(at 121.92 129.54 0)
 			(effects
 				(font
@@
 		)
 		(property "Description" "coaxial connector (BNC, SMA, SMB, SMC, Cinch/RCA, LEMO, ...)"
-			(at 109.22 129.54 0)
+			(at 121.92 129.54 0)
 			(effects
 				(font
@@
 	(symbol
 		(lib_id "Connector:Conn_Coaxial")
-		(at 109.22 157.48 0)
+		(at 120.65 157.48 0)
 		(unit 1)
 		(exclude_from_sim no)
@@
 		(dnp no)
 		(property "Reference" "J18"
-			(at 113.03 156.5031 0)
+			(at 124.46 156.5031 0)
 			(effects
 				(font
@@
 		)
 		(property "Value" "Conn_Coaxial"
-			(at 113.03 159.0431 0)
+			(at 124.46 159.0431 0)
 			(effects
 				(font
@@
 		)
 		(property "Footprint" "Connector_Coaxial:U.FL_Hirose_U.FL-R-SMT-1_Vertical"
-			(at 109.22 157.48 0)
+			(at 120.65 157.48 0)
 			(effects
 				(font
@@
 		)
 		(property "Datasheet" "~"
-			(at 109.22 157.48 0)
+			(at 120.65 157.48 0)
 			(effects
 				(font
@@
 		)
 		(property "Description" "coaxial connector (BNC, SMA, SMB, SMC, Cinch/RCA, LEMO, ...)"
-			(at 109.22 157.48 0)
+			(at 120.65 157.48 0)
 			(effects
 				(font
