File: 4phaseshift/Vector_Modulator_TestBoard.kicad_sch (KiCad schematic)
At the start: 20 parts, among them J7 Conn_Coaxial, U10 TLV2372, U11 ADL5375-15ACPZ-WP

Commit message: gerbers generated for 4 element
Connections:
- net VCC renamed LocalVCC
Other:
- sheet Amplifier_SBB5089Z ports: added LocalVCC; removed none

Commit message: updated resistor values
Parts:
- R5, R6, R7, R8: value 100k -> 10k
Changed lines of the file:
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@@
 			)
 		)
-		(property "Value" "100k"
+		(property "Value" "10k"
 			(at 100.33 78.74 90)
 			(effects
@@
 			)
 		)
-		(property "Value" "100k"
+		(property "Value" "10k"
 			(at 102.87 105.41 90)
 			(effects
@@
 			)
 		)
-		(property "Value" "100k"
+		(property "Value" "10k"
 			(at 88.9 96.52 90)
 			(effects
@@
 			)
 		)
-		(property "Value" "100k"
+		(property "Value" "10k"
 			(at 86.36 69.85 90)
 			(effects
