File: 4phaseshift/4phaseshift.kicad_pcb (KiCad board)
At the start: 4 copper layers, 61 x 70 mm, 135 parts, among them J1 Conn_Coaxial, J10 Conn_Coaxial, J2 Conn_01x05_Pin, J3 Conn_Coaxial, J4 Conn_Coaxial, J7 Conn_Coaxial, J8 Conn_Coaxial, J9 Conn_Coaxial, U1 AMS1117, U10 TLV2372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

Commit message: gerbers generated for 4 element
Parts:
- removed TP1, TP2: TestPoint, Connector_PinHeader_2.54mm:PinHeader_1x01_P2.54mm_Vertical
- added C6: 10u, Capacitor_SMD:C_0603_1608Metric_Pad1.08x0.95mm_HandSolder, B.Cu at (125.1, 168.5)
- added C7: 10u, Capacitor_SMD:C_0603_1608Metric_Pad1.08x0.95mm_HandSolder, B.Cu at (125.1, 165.5)
- added C9: 1u, Capacitor_SMD:C_0603_1608Metric_Pad1.08x0.95mm_HandSolder, B.Cu at (125.1, 167.0)
- added GND: TestPoint, Connector_PinHeader_2.54mm:PinHeader_1x01_P2.54mm_Vertical, B.Cu at (134.2, 168.2)
- added R23: 300, Resistor_SMD:R_0603_1608Metric_Pad0.98x0.95mm_HandSolder, B.Cu at (125.1, 162.5)
- added R24: 100, Resistor_SMD:R_0603_1608Metric_Pad0.98x0.95mm_HandSolder, B.Cu at (125.1, 164.0)
- added U2: AMS1117, Package_TO_SOT_SMD:SOT-223-3_TabPin2, B.Cu at (118.9, 165.6)
- added VS: TestPoint, Connector_PinHeader_2.54mm:PinHeader_1x01_P2.54mm_Vertical, B.Cu at (130.4, 168.2)
- J2: moved to B.Cu
- moved U1 13.4 mm to (104.9, 165.6)
- moved C1 13.4 mm to (111.1, 168.5)
- moved C2 13.4 mm to (111.1, 165.5)
- moved R1 13.4 mm to (111.1, 162.5)
- moved R2 13.4 mm to (111.1, 164.0)
- moved C3 13.4 mm to (111.1, 167.0)
- turned J2 to 180 degrees
Connections:
- net Net-(J2-Pin_3) renamed /LDAC
- net Net-(J2-Pin_4) renamed /SCL
- C18 pad 2: VCC -> VCC2
- C19 pad 2: VCC -> VCC2
- C20 pad 2: VCC -> VCC2
- C44 pad 2: VCC -> VCC2
- C46 pad 2: VCC -> VCC2
- C47 pad 1: VCC -> VCC2
- C48 pad 1: VCC -> VCC2
- C49 pad 1: VCC -> VCC2
- C53 pad 2: VCC -> VCC2
- C54 pad 2: VCC -> VCC2
- C55 pad 2: VCC -> VCC2
- C57 pad 2: VCC -> VCC2
- C59 pad 2: VCC -> VCC2
- C60 pad 1: VCC -> VCC2
- C61 pad 1: VCC -> VCC2
- C62 pad 1: VCC -> VCC2
- C66 pad 2: VCC -> VCC2
- C67 pad 2: VCC -> VCC2
- C68 pad 2: VCC -> VCC2
- L2 pad 1: VCC -> VCC2
- L4 pad 1: VCC -> VCC2
- L5 pad 1: VCC -> VCC2
- R32 pad 1: VCC -> VCC2
- R34 pad 1: VCC -> VCC2
- RV1 pad 3: VCC -> VCC2
- U15 pad 8: VCC -> VCC2
- U16 pad 18: VCC -> VCC2
- U16 pad 24: VCC -> VCC2
- U18 pad 8: VCC -> VCC2
- U19 pad 18: VCC -> VCC2
- U19 pad 24: VCC -> VCC2
- U3 pad 7: VCC -> VCC2
Routing:
- net VCC2: track 0.00 -> 193.9 mm, vias 0 -> 11
- net VCC: track 331.6 -> 187.0 mm, vias 17 -> 10
- net VS: track 7.16 -> 43.6 mm, vias 0 -> 4
- net GND: track 153.9 -> 163.6 mm, vias 20 -> 30
- net Net-(U2-ADJ): track 0.00 -> 3.93 mm
Other:
- board text added: "2V5"
- board text added: "GND"
- board text added: "LDAC"
- board text added: "SCL"
- board text added: "SDA"

Commit message: saatvik mad
Parts:
- L1, L2, L3, L4, L5: value 82n -> 20n
- R1, R23: value 300 -> 560
- R10, R11, R12, R13, R14, R15, R16, R17, R18, R19, R20, R5, R6, R7, R8, R9: value 100k -> 10k
- R2, R24: value 100 -> 187
